Commit message: adding diagnostics

File: sphero_description/urdf/sphero.urdf (robot description, URDF)
Before this commit: robot sphero, 2 links, 1 joints
Links:
- link base_link: geometry collision sphere radius=0.04; visual mesh filename=package://sphero_description/meshes/Sphero.dae scale=0.0254 0.0254 0.0254

Commit message: adding textured sphero

File: sphero_description/urdf/sphero.urdf (robot description, URDF)
Before this commit: robot sphero, 2 links, 1 joints
Links:
- link base_footprint: geometry 
- link base_link: geometry collision sphere radius=0.0381; visual mesh filename=package://sphero_description/meshes/Sphero_Textured.dae scale=0.0127 0.0127 0.0127
Joints:
- joint base_footprint_joint: child base_link -> base_footprint; origin xyz=0 0 0.02 rpy=0 0 0 -> xyz=0 0 -0.0381 rpy=0 0 0; parent base_footprint -> base_link

Commit message: updating urdf to launch correctly

File: sphero_description/urdf/sphero.urdf (robot description, URDF)
Before this commit: robot sphero, 2 links, 1 joints
Links:
- link base_footprint: mass 0.0 -> None
Joints:
- joint base_footprint_joint: child base_footprint -> base_link; origin xyz=0 0 -0.0381 rpy=0 0 0 -> xyz=0 0 0.0381 rpy=0 0 0; parent base_link -> base_footprint
